Commit message: fix elbow joint limit

File: pal_sea_arm_description/urdf/arm/arm_properties/arm_tiago-pro.properties.xacro (robot description, xacro)
@@ -52,5 +52,5 @@
 </xacro:macro>
 <xacro:macro name="origin_joint_3" params="reflect">
-        <origin xyz="-0.15 -0.02 0" rpy="3.1415 1.5707 0" />
+    <origin xyz="-0.15 -0.02 0" rpy="3.1415 1.5707 0" />
 </xacro:macro>
 <xacro:macro name="inertial_link_4" params="reflect">

File: pal_sea_arm_description/urdf/arm/limits/arm_tiago-pro.limits.xacro (robot description, xacro)
@@ -11,6 +11,6 @@
   <xacro:property name="arm_3_joint_ub" value="148.97" />
   <xacro:property name="arm_3_joint_lb" value="-148.97" />
-  <xacro:property name="arm_4_joint_ub" value="139.8" />
-  <xacro:property name="arm_4_joint_lb" value="-63.03" />
+  <xacro:property name="arm_4_joint_ub" value="63.03" />
+  <xacro:property name="arm_4_joint_lb" value="-139.8" />
   <xacro:property name="arm_5_joint_ub" value="148.97" />
   <xacro:property name="arm_5_joint_lb" value="-148.97" />
