Commit message: Update joint limit for joint 7 tiago pro

File: pal_sea_arm_description/urdf/arm/limits/arm_tiago-pro.limits.xacro (robot description, xacro)
@@ -17,6 +17,6 @@
   <xacro:property name="arm_6_joint_ub" value="114.59" />
   <xacro:property name="arm_6_joint_lb" value="-114.59" />
-  <xacro:property name="arm_7_joint_ub" value="148.97" />
-  <xacro:property name="arm_7_joint_lb" value="-148.97" />
+  <xacro:property name="arm_7_joint_ub" value="139.8" />
+  <xacro:property name="arm_7_joint_lb" value="-139.8" />
   <xacro:property name="arm_1_max_velocity"      value="1.95" />
   <xacro:property name="arm_2_max_velocity"      value="1.95" />
