Commit message: add pal_atc package

File: pal_sea_arm_description/urdf/end_effector/end_effector.urdf.xacro (robot description, xacro)
@@ -27,4 +27,11 @@
         <origin xyz="0.0 0.0 0.0" rpy="0 0 0"/>
       </xacro:pal_pro_gripper>
+    </xacro:if>
+    <!-- PAL ATC -->
+    <xacro:if value="${type == 'pal-atc'}">
+      <xacro:include filename="$(find pal_atc_description)/urdf/gripper.urdf.xacro" />
+      <xacro:pal_atc name="${name}" parent="${parent}" tool_changer="${tool_changer}">
+        <origin xyz="0.0 0.0 0.0" rpy="0 0 0"/>
+      </xacro:pal_atc>
     </xacro:if>
   <!--Allegro Hand-->
