Commit message: reducing max velocity for prevent ethercat problem

File: pal_sea_arm_description/urdf/arm/arm_limits/pal-sea-arm-standalone/arm.limits.xacro (robot description, xacro)
@@ -11,8 +11,8 @@
   <xacro:property name="arm_4_joint_lb" value="-139.8" />
   <!-- Velocity limits -->
-  <xacro:property name="arm_1_max_velocity" value="1.95" />
-  <xacro:property name="arm_2_max_velocity" value="1.95" />
-  <xacro:property name="arm_3_max_velocity" value="3.95" />
-  <xacro:property name="arm_4_max_velocity" value="3.95" />
+  <xacro:property name="arm_1_max_velocity" value="1.36" /> <!-- ATTENTION -->
+  <xacro:property name="arm_2_max_velocity" value="1.36" /> <!-- Limits -->
+  <xacro:property name="arm_3_max_velocity" value="2.76" /> <!-- reduced by -->
+  <xacro:property name="arm_4_max_velocity" value="2.76" /> <!-- 30 % -->
   <!-- Effort limits -->
   <xacro:property name="arm_1_max_effort" value="43.0" />
