Commit message: Proper launch of the RH8D hand
Removes the mimic flag and properly loads the topic based system (used
for the HW hand)

File: pal_sea_arm_description/urdf/end_effector/humanoid/rh8d_hand.urdf.xacro (robot description, xacro)
@@ -20,5 +20,5 @@
     - reflect: Set to 1 for a right end effector, or to -1 for a left end effector
   -->
-  <xacro:macro name="hand" params="name parent side mimic:=False *origin">
+  <xacro:macro name="hand" params="name parent side *origin">
     <!-- PROPERTIES -->
     <xacro:property name="reflect" value="${'1' if side == 'left' else '-1'}" />
@@ -26,5 +26,5 @@
     <xacro:include filename="$(find rh8d_description)/urdf/hand/hand.urdf.xacro"/>
     <!-- ROBOT DEFINITION -->
-    <xacro:rh8d_hand name="${name}" side="${side}" reflect="${reflect}" parent="${parent}" mimic="${mimic}" >
+    <xacro:rh8d_hand name="${name}" side="${side}" reflect="${reflect}" parent="${parent}" >
       <xacro:insert_block name="origin"/>
     </xacro:rh8d_hand>

File: pal_sea_arm_description/urdf/end_effector/humanoid/ros2_control.urdf.xacro (robot description, xacro)
@@ -15,11 +15,22 @@
   <!-- MACRO DEFINITION-->
   <xacro:macro name="end_effector_ros2_control" params="side end_effector_type">
-    <xacro:if value="${end_effector_${side} == 'gripper'}">
+    <xacro:if value="${end_effector_type == 'gripper'}">
       <xacro:include filename="$(find pal_pro_gripper_description)/urdf/gripper.ros2_control.xacro" />
       <xacro:ros2_control_pal_pro_gripper name="gripper_${side}" reduction="1.0"  sim_type="${sim_type}"/>
     </xacro:if>
-    <xacro:if value="${end_effector_${side} == 'RH8D'}">
+    <!-- RH8D on real hardware is driven by rh8d_topic_driver, which needs its own
+         <ros2_control> element with the topic-based plugin. That cannot be nested here, so it
+         is emitted alongside the main system block by end_effector_standalone_ros2_control. -->
+    <xacro:if value="${end_effector_type == 'RH8D' and sim_type != 'no-simulation'}">
       <xacro:include filename="$(find rh8d_description)/urdf/hand/ros2_control.urdf.xacro" />
-      <xacro:hand_ros2_control side="${side}" mimic="${use_mimic}"/>
+      <xacro:hand_ros2_control side="${side}"/>
+    </xacro:if>
+  </xacro:macro>
+  <!-- End effectors that bring their own <ros2_control> element. Must be instantiated OUTSIDE
+       the robot's main system block. -->
+  <xacro:macro name="end_effector_standalone_ros2_control" params="side end_effector_type">
+    <xacro:if value="${end_effector_type == 'RH8D' and sim_type == 'no-simulation'}">
+      <xacro:include filename="$(find rh8d_description)/ros2_control/topic_based_ros2_control.urdf.xacro" />
+      <xacro:rh8d_topic_based_ros2_control side="${side}"/>
     </xacro:if>
   </xacro:macro>
